File: C_Fabrication/V0/A_Circuit/A_Kicad/Self_Balancing_Bot_V0/Self_Balancing_Bot_V0.kicad_pcb (KiCad board)
At the start: 4 copper layers, 90 x 59 mm, 18 parts, among them J2 Conn_01x04_Pin, J3 Conn_01x04_Pin, J4 Screw_Terminal_01x02, SW1 SW_SPDT, U5 TSR1-2450E

Commit message: Electronic design redaction, Annexes
Parts:
- R3: value R -> 61k
- R4: value R -> 10k
Changed lines of the file:
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@@
 			(crossoutdnponfab yes)
 			(subtractmaskfromsilk no)
-			(outputformat 1)
+			(outputformat 4)
 			(mirror no)
 			(drillshape 0)
 			(scaleselection 1)
-			(outputdirectory "../Gerbers/")
+			(outputdirectory "../../../../../A_Documentation/Rapport/assets/figures/")
 		)
 	)
@@
 		)
 		(sheetname "/")
-		(sheetfile "Balance_bot_V0.kicad_sch")
+		(sheetfile "Self_Balancing_Bot_V0.kicad_sch")
 		(attr through_hole)
 		(fp_rect
@@
 		(property ki_fp_filters "C_*")
 		(sheetname "/")
-		(sheetfile "Balance_bot_V0.kicad_sch")
+		(sheetfile "Self_Balancing_Bot_V0.kicad_sch")
 		(attr smd)
 		(fp_line
@@
 			)
 		)
-		(property "Value" "R"
+		(property "Value" "61k"
 			(at 0 1.83 90)
 			(layer "F.Fab")
@@
 		(property ki_fp_filters "R_*")
 		(sheetname "/")
-		(sheetfile "Balance_bot_V0.kicad_sch")
+		(sheetfile "Self_Balancing_Bot_V0.kicad_sch")
 		(attr smd)
 		(fp_line
@@
 		)
 		(sheetname "/")
-		(sheetfile "Balance_bot_V0.kicad_sch")
+		(sheetfile "Self_Balancing_Bot_V0.kicad_sch")
 		(attr through_hole)
 		(fp_line
@@
 		(property ki_fp_filters "R_*")
 		(sheetname "/")
-		(sheetfile "Balance_bot_V0.kicad_sch")
+		(sheetfile "Self_Balancing_Bot_V0.kicad_sch")
 		(attr smd)
 		(fp_line
@@
 		)
 		(sheetname "/")
-		(sheetfile "Balance_bot_V0.kicad_sch")
+		(sheetfile "Self_Balancing_Bot_V0.kicad_sch")
 		(attr through_hole)
 		(fp_line
@@
 		(property ki_fp_filters "Connector*:*_1x??_*")
 		(sheetname "/")
-		(sheetfile "Balance_bot_V0.kicad_sch")
+		(sheetfile "Self_Balancing_Bot_V0.kicad_sch")
 		(attr through_hole)
 		(fp_line
@@
 		(property ki_fp_filters "Connector*:*_1x??_*")
 		(sheetname "/")
-		(sheetfile "Balance_bot_V0.kicad_sch")
+		(sheetfile "Self_Balancing_Bot_V0.kicad_sch")
 		(attr through_hole)
 		(fp_line
@@
 		)
 		(sheetname "/")
-		(sheetfile "Balance_bot_V0.kicad_sch")
+		(sheetfile "Self_Balancing_Bot_V0.kicad_sch")
 		(attr through_hole)
 		(fp_line
@@
 		)
 		(sheetname "/")
-		(sheetfile "Balance_bot_V0.kicad_sch")
+		(sheetfile "Self_Balancing_Bot_V0.kicad_sch")
 		(attr through_hole)
 		(fp_rect
@@
 		(property ki_fp_filters "TerminalBlock*:*")
 		(sheetname "/")
-		(sheetfile "Balance_bot_V0.kicad_sch")
+		(sheetfile "Self_Balancing_Bot_V0.kicad_sch")
 		(attr through_hole)
 		(fp_line
@@
 		(property ki_fp_filters "Converter*DCDC*TRACO*TSR1*xxxxE*THT*")
 		(sheetname "/")
-		(sheetfile "Balance_bot_V0.kicad_sch")
+		(sheetfile "Self_Balancing_Bot_V0.kicad_sch")
 		(attr through_hole)
 		(fp_line
@@
 			)
 		)
-		(property "Value" "R"
+		(property "Value" "10k"
 			(at 0 1.83 90)
 			(layer "F.Fab")
@@
 		(property ki_fp_filters "R_*")
 		(sheetname "/")
-		(sheetfile "Balance_bot_V0.kicad_sch")
+		(sheetfile "Self_Balancing_Bot_V0.kicad_sch")
 		(attr smd)
 		(fp_line
@@
 		(property ki_fp_filters "C_*")
 		(sheetname "/")
-		(sheetfile "Balance_bot_V0.kicad_sch")
+		(sheetfile "Self_Balancing_Bot_V0.kicad_sch")
 		(attr smd)
 		(fp_line
@@
 		(layer "User.1")
 		(pts
+			(xy 188 74) (xy 187.75 125)
+		)
+		(height 14.75)
+		(orientation 1)
+		(format
+			(prefix "")
+			(suffix "")
+			(units 3)
+			(units_format 0)
+			(precision 4)
+			(suppress_zeroes yes)
+		)
+		(style
+			(thickness 0.1)
+			(arrow_length 1.27)
+			(text_position_mode 0)
+			(arrow_direction outward)
+			(extension_height 0.58642)
+			(extension_offset 0.5)
+			(keep_text_aligned yes)
+		)
+		(gr_text "51"
+			(at 201.6 99.5 90)
+			(layer "User.1")
+			(effects
+				(font
+					(size 1 1)
+					(thickness 0.15)
+				)
+			)
+		)
+	)
+	(dimension
+		(type orthogonal)
+		(layer "User.1")
+		(pts
 			(xy 192 70) (xy 193.5 129)
 		)
@@
 			(layer "User.1")
 			(effects
+				(font
+					(size 1 1)
+					(thickness 0.15)
+				)
+			)
+		)
+	)
+	(dimension
+		(type orthogonal)
+		(layer "User.1")
+		(pts
+			(xy 188 74) (xy 106 74)
+		)
+		(height -9.5)
+		(orientation 0)
+		(format
+			(prefix "")
+			(suffix "")
+			(units 3)
+			(units_format 0)
+			(precision 4)
+			(suppress_zeroes yes)
+		)
+		(style
+			(thickness 0.1)
+			(arrow_length 1.27)
+			(text_position_mode 0)
+			(arrow_direction outward)
+			(extension_height 0.58642)
+			(extension_offset 0.5)
+			(keep_text_aligned yes)
+		)
+		(gr_text "82"
+			(at 147 63.35 0)
+			(layer "User.1")
+			(effects
