File: C_Fabrication/V0/A_Circuit/A_Kicad/Self_Balancing_Bot_V0/Self_Balancing_Bot_V0.kicad_sch (KiCad schematic)
At the start: 14 parts, among them J2 Conn_01x04_Pin, J3 Conn_01x04_Pin, J4 Screw_Terminal_01x02, SW1 SW_SPDT, U5 TSR1-2450E

Commit message: Electronic design redaction, Annexes
Other:
- company: (none) -> Ding Jérémy
- title: (none) -> Self_Balancing_Bot_V0
Changed lines of the file:
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@@
 	(generator_version "9.0")
 	(paper "A4")
+	(title_block
+		(title "Self_Balancing_Bot_V0")
+		(date "21/04/2026")
+		(rev "V0")
+		(company "Ding Jérémy")
+	)
 	(rectangle
 		(start 205.74 40.64)

Commit message: End of electronic design's rapport
Parts:
- R3: value 61k -> 51k
Changed lines of the file:
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@@
 			)
 		)
-		(property "Value" "61k"
+		(property "Value" "51k"
 			(at 72.644 160.02 0)
 			(effects
